File: hardware/ROBOBIKE05_PCBA/ROBOBIKE05_PCBA.kicad_sch (KiCad schematic)
At the start: 53 parts, among them J1 3P PIN HEADER, J10 2.54, J11 WIRING HOLE, J2 3P PIN HEADER, J3 3P PIN HEADER, J4 PINHEADER, J5 2.54, J6 SM-2P, J7 SM-2R, J8 2.54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

Commit message: use external Interrupt
Other:
- note added: "IO20 IO21 3V3 GND SOLDER CONNECT"
- note removed: "IO20 IO21 IO0 GND SOLDER CONNECT"
Changed lines of the file:
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@@
 		)
 	)
-	(text "IO20\nIO21\nIO0\nGND\n\nSOLDER CONNECT"
+	(text "IO20\nIO21\n3V3\nGND\n\nSOLDER CONNECT"
 		(exclude_from_sim no)
 		(at 22.225 173.99 0)
